File: schematic/MegaBlaster2.kicad_sch (KiCad schematic)
At the start: 118 parts, among them J1 USB_B, J2 SWD, J3 Micro_SD_Card, J4 AudioJack3, SW2 SW_Push_Dual, SW3 SW_Push_Dual, SW4 SW_Push_Dual, SW5 SW_Push_Dual, SW6 SW_Push_Dual, SW7 SW_Push_Dual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

Commit message: footprints
Parts:
- removed TP7: DAC0, symbol Connector:TestPoint
- removed TP8: DAC1, symbol Connector:TestPoint
- added J5: DAC_Enable, Connector_PinHeader_2.54mm:PinHeader_2x03_P2.54mm_Vertical, symbol Connector_Generic:Conn_02x03_Odd_Even
- added R30, R31: 10K, Resistor_SMD:R_0805_2012Metric, symbol Device:R_Small
- RV1, RV2, RV3: footprint (none) -> Potentiometer_THT:Potentiometer_Alps_RK097_Dual_Horizontal
- TP2, TP3: footprint (none) -> TestPoint:TestPoint_Pad_D2.0mm
- U11: footprint (none) -> Package_DIP:DIP-24_W15.24mm_Socket
- U7, U9: footprint (none) -> Package_SO:SOIC-14_3.9x8.7mm_P1.27mm
- U8: footprint (none) -> Package_DIP:DIP-16_W7.62mm_Socket
Connections:
- net DAC0: now also J5.2 (Pin_2); no longer C39.2
- net DAC1: now also J5.1 (Pin_1); no longer C43.2
- net GND: now also R30.2, R31.2
- new net: J5.6 (Pin_6), R31.1
- new net: C43.2, J5.3 (Pin_3)
- new net: C39.2, J5.4 (Pin_4)
- new net: J5.5 (Pin_5), R30.1
Other:
- moved on the sheet: C26, C39, C40, C41, C42, C43, C44, C45, C46, R17, R20, R21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

Commit message: PCB first pass
Connections:
- net D0: now also U1.35 (PA16); no longer U1.44 (PA23)
- net D1: now also U1.36 (PA17); no longer U1.43 (PA22)
- net D2: now also U1.37 (PA18); no longer U1.42 (PA21)
- net D3: now also U1.38 (PA19); no longer U1.41 (PA20)
- net D4: now also U1.41 (PA20); no longer U1.38 (PA19)
- net D5: now also U1.42 (PA21); no longer U1.37 (PA18)
- net D6: now also U1.43 (PA22); no longer U1.36 (PA17)
- net D7: now also U1.44 (PA23); no longer U1.35 (PA16)
Changed lines of the file:
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@@
     (effects (font (size 1.27 1.27)) (justify left bottom))
   )
-  (global_label "D7" (shape input) (at 52.07 87.63 180) (fields_autoplaced)
-    (effects (font (size 1.27 1.27)) (justify right))
-    (property "Intersheet References" "${INTERSHEET_REFS}" (id 0) (at 0 0 0)
+  (global_label "D7" (shape input) (at 52.07 105.41 180) (fields_autoplaced)
+    (effects (font (size 1.27 1.27)) (justify right))
+    (property "Intersheet References" "${INTERSHEET_REFS}" (id 0) (at 0 193.04 0)
       (effects (font (size 1.27 1.27)) hide)
     )
@@
     )
   )
-  (global_label "D4" (shape input) (at 52.07 95.25 180) (fields_autoplaced)
-    (effects (font (size 1.27 1.27)) (justify right))
-    (property "Intersheet References" "${INTERSHEET_REFS}" (id 0) (at 0 0 0)
+  (global_label "D4" (shape input) (at 52.07 97.79 180) (fields_autoplaced)
+    (effects (font (size 1.27 1.27)) (justify right))
+    (property "Intersheet References" "${INTERSHEET_REFS}" (id 0) (at 0 193.04 0)
       (effects (font (size 1.27 1.27)) hide)
     )
@@
     )
   )
-  (global_label "D2" (shape input) (at 52.07 100.33 180) (fields_autoplaced)
-    (effects (font (size 1.27 1.27)) (justify right))
-    (property "Intersheet References" "${INTERSHEET_REFS}" (id 0) (at 0 0 0)
+  (global_label "D2" (shape input) (at 52.07 92.71 180) (fields_autoplaced)
+    (effects (font (size 1.27 1.27)) (justify right))
+    (property "Intersheet References" "${INTERSHEET_REFS}" (id 0) (at 0 193.04 0)
       (effects (font (size 1.27 1.27)) hide)
     )
@@
     )
   )
-  (global_label "D5" (shape input) (at 52.07 92.71 180) (fields_autoplaced)
-    (effects (font (size 1.27 1.27)) (justify right))
-    (property "Intersheet References" "${INTERSHEET_REFS}" (id 0) (at 0 0 0)
+  (global_label "D5" (shape input) (at 52.07 100.33 180) (fields_autoplaced)
+    (effects (font (size 1.27 1.27)) (justify right))
+    (property "Intersheet References" "${INTERSHEET_REFS}" (id 0) (at 0 193.04 0)
       (effects (font (size 1.27 1.27)) hide)
     )
@@
     )
   )
-  (global_label "D3" (shape input) (at 52.07 97.79 180) (fields_autoplaced)
-    (effects (font (size 1.27 1.27)) (justify right))
-    (property "Intersheet References" "${INTERSHEET_REFS}" (id 0) (at 0 0 0)
+  (global_label "D3" (shape input) (at 52.07 95.25 180) (fields_autoplaced)
+    (effects (font (size 1.27 1.27)) (justify right))
+    (property "Intersheet References" "${INTERSHEET_REFS}" (id 0) (at 0 193.04 0)
       (effects (font (size 1.27 1.27)) hide)
     )
@@
     )
   )
-  (global_label "D6" (shape input) (at 52.07 90.17 180) (fields_autoplaced)
-    (effects (font (size 1.27 1.27)) (justify right))
-    (property "Intersheet References" "${INTERSHEET_REFS}" (id 0) (at 0 0 0)
-      (effects (font (size 1.27 1.27)) hide)
-    )
-  )
-  (global_label "D0" (shape input) (at 52.07 105.41 180) (fields_autoplaced)
-    (effects (font (size 1.27 1.27)) (justify right))
-    (property "Intersheet References" "${INTERSHEET_REFS}" (id 0) (at 0 0 0)
+  (global_label "D6" (shape input) (at 52.07 102.87 180) (fields_autoplaced)
+    (effects (font (size 1.27 1.27)) (justify right))
+    (property "Intersheet References" "${INTERSHEET_REFS}" (id 0) (at 0 193.04 0)
+      (effects (font (size 1.27 1.27)) hide)
+    )
+  )
+  (global_label "D0" (shape input) (at 52.07 87.63 180) (fields_autoplaced)
+    (effects (font (size 1.27 1.27)) (justify right))
+    (property "Intersheet References" "${INTERSHEET_REFS}" (id 0) (at 0 193.04 0)
       (effects (font (size 1.27 1.27)) hide)
     )
@@
     )
   )
-  (global_label "D1" (shape input) (at 52.07 102.87 180) (fields_autoplaced)
-    (effects (font (size 1.27 1.27)) (justify right))
-    (property "Intersheet References" "${INTERSHEET_REFS}" (id 0) (at 0 0 0)
-      (effects (font (size 1.27 1.27)) hide)
-    )
+  (global_label "D1" (shape input) (at 52.07 90.17 180) (fields_autoplaced)
+    (effects (font (size 1.27 1.27)) (justify right))
+    (property "Intersheet References" "${INTERSHEET_REFS}" (id 0) (at 0 193.04 0)
+      (effects (font (size 1.27 1.27)) hide)
+    )

Commit message: 2M resistor update
Parts:
- added R32, R33: 2M, Resistor_SMD:R_0805_2012Metric, symbol Device:R_Small
- U7: value TL074 -> MCP6004
Connections:
- net GND: now also R32.2, R33.2
- net at C40.1, R17.2, U9.3 (+): now also R32.1
- net at C44.1, R24.2, U9.5 (+): now also R33.1
Other:
- moved on the sheet: R24
Changed lines of the file:
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@@
   (junction (at 347.98 199.39) (diameter 0) (color 0 0 0 0)
   )
+  (junction (at 307.34 116.84) (diameter 0) (color 0 0 0 0)
+  )
   (junction (at 394.97 20.32) (diameter 0) (color 0 0 0 0)
   )
@@
   (junction (at 393.7 128.27) (diameter 0) (color 0 0 0 0)
   )
-  (junction (at 307.34 116.84) (diameter 0) (color 0 0 0 0)
-  )
   (junction (at 365.76 184.15) (diameter 0) (color 0 0 0 0)
   )
@@
     (stroke (width 0) (type default) (color 0 0 0 0))
   )
-  (wire (pts (xy 307.34 116.84) (xy 311.15 116.84))
+  (wire (pts (xy 303.53 116.84) (xy 307.34 116.84))
     (stroke (width 0) (type default) (color 0 0 0 0))
   )
@@
     (stroke (width 0) (type default) (color 0 0 0 0))
   )
-  (wire (pts (xy 307.34 114.3) (xy 307.34 116.84))
-    (stroke (width 0) (type default) (color 0 0 0 0))
-  )
   (wire (pts (xy 313.69 67.31) (xy 313.69 71.12))
     (stroke (width 0) (type default) (color 0 0 0 0))
@@
     (stroke (width 0) (type default) (color 0 0 0 0))
   )
-  (wire (pts (xy 303.53 116.84) (xy 307.34 116.84))
-    (stroke (width 0) (type default) (color 0 0 0 0))
-  )
   (wire (pts (xy 394.97 20.32) (xy 398.78 20.32))
     (stroke (width 0) (type default) (color 0 0 0 0))
@@
     (stroke (width 0) (type default) (color 0 0 0 0))
   )
+  (wire (pts (xy 307.34 116.84) (xy 311.15 116.84))
+    (stroke (width 0) (type default) (color 0 0 0 0))
+  )
   (wire (pts (xy 383.54 191.77) (xy 383.54 187.96))
     (stroke (width 0) (type default) (color 0 0 0 0))
@@
     (in_bom yes) (on_board yes)
     (property "Reference" "U7" (id 0) (at 325.12 17.78 0))
-    (property "Value" "TL074" (id 1) (at 326.39 20.32 0))
+    (property "Value" "MCP6004" (id 1) (at 326.39 20.32 0))
     (property "Footprint" "Package_SO:SOIC-14_3.9x8.7mm_P1.27mm" (id 2) (at 320.04 20.32 0)
       (effects (font (size 1.27 1.27)) hide)
@@
     (pin "1")
   )
+  (symbol (lib_id "Device:R_Small") (at 307.34 99.06 0) (unit 1)
+    (in_bom yes) (on_board yes)
+    (property "Reference" "R32" (id 0) (at 304.8 97.79 0))
+    (property "Value" "2M" (id 1) (at 304.8 100.33 0))
+    (property "Footprint" "Resistor_SMD:R_0805_2012Metric" (id 2) (at 307.34 99.06 0)
+      (effects (font (size 1.27 1.27)) hide)
+    )
+    (property "Datasheet" "~" (id 3) (at 307.34 99.06 0)
+      (effects (font (size 1.27 1.27)) hide)
+    )
+    (pin "1")
+    (pin "2")
+  )
   (symbol (lib_id "Device:R_Small") (at 365.76 54.61 90) (unit 1)
     (in_bom yes) (on_board yes)
@@
     (pin "2")
   )
-  (symbol (lib_id "Device:R_Small") (at 307.34 111.76 0) (unit 1)
+  (symbol (lib_id "Device:R_Small") (at 307.34 114.3 0) (unit 1)
     (in_bom yes) (on_board yes)
-    (property "Reference" "R24" (id 0) (at 309.88 109.22 0))
-    (property "Value" "1M" (id 1) (at 309.88 111.76 0))
-    (property "Footprint" "Resistor_SMD:R_0805_2012Metric" (id 2) (at 307.34 111.76 0)
+    (property "Reference" "R24" (id 0) (at 309.88 111.76 0))
+    (property "Value" "1M" (id 1) (at 309.88 114.3 0))
+    (property "Footprint" "Resistor_SMD:R_0805_2012Metric" (id 2) (at 307.34 114.3 0)
       (effects (font (size 1.27 1.27)) hide)
     )
-    (property "Datasheet" "~" (id 3) (at 307.34 111.76 0)
+    (property "Datasheet" "~" (id 3) (at 307.34 114.3 0)
       (effects (font (size 1.27 1.27)) hide)
     )
@@
     (pin "2")
   )
-  (symbol (lib_id "power:+2V5") (at 307.34 109.22 0) (unit 1)
-    (in_bom yes) (on_board yes) (fields_autoplaced)
-    (property "Reference" "#PWR0126" (id 0) (at 307.34 113.03 0)
+  (symbol (lib_id "power:+2V5") (at 307.34 111.76 0) (unit 1)
+    (in_bom yes) (on_board yes)
+    (property "Reference" "#PWR0126" (id 0) (at 307.34 115.57 0)
       (effects (font (size 1.27 1.27)) hide)
     )
-    (property "Value" "+2V5" (id 1) (at 307.34 105.6155 0))
-    (property "Footprint" "" (id 2) (at 307.34 109.22 0)
+    (property "Value" "+2V5" (id 1) (at 307.34 107.95 0))
+    (property "Footprint" "" (id 2) (at 307.34 111.76 0)
       (effects (font (size 1.27 1.27)) hide)
     )
-    (property "Datasheet" "" (id 3) (at 307.34 109.22 0)
+    (property "Datasheet" "" (id 3) (at 307.34 111.76 0)
       (effects (font (size 1.27 1.27)) hide)
     )
@@
     (in_bom yes) (on_board yes)
     (property "Reference" "U7" (id 0) (at 325.12 59.69 0))
-    (property "Value" "TL074" (id 1) (at 326.39 62.23 0))
+    (property "Value" "MCP6004" (id 1) (at 326.39 62.23 0))
     (property "Footprint" "Package_SO:SOIC-14_3.9x8.7mm_P1.27mm" (id 2) (at 320.04 62.23 0)
       (effects (font (size 1.27 1.27)) hide)
@@
       (effects (font (size 1.27 1.27)) (justify left))
     )
-    (property "Value" "TL074" (id 1) (at 387.35 30.48 0)
+    (property "Value" "MCP6004" (id 1) (at 387.35 30.48 0)
       (effects (font (size 1.27 1.27)) (justify left))
     )
@@
     (pin "4")
   )
+  (symbol (lib_id "Device:R_Small") (at 307.34 119.38 0) (unit 1)
+    (in_bom yes) (on_board yes)
+    (property "Reference" "R33" (id 0) (at 304.8 118.11 0))
+    (property "Value" "2M" (id 1) (at 304.8 120.65 0))
+    (property "Footprint" "Resistor_SMD:R_0805_2012Metric" (id 2) (at 307.34 119.38 0)
+      (effects (font (size 1.27 1.27)) hide)
+    )
+    (property "Datasheet" "~" (id 3) (at 307.34 119.38 0)
+      (effects (font (size 1.27 1.27)) hide)
+    )
+    (pin "1")
+    (pin "2")
+  )
   (symbol (lib_id "power:+5V") (at 219.71 99.06 90) (unit 1)
     (in_bom yes) (on_board yes)
@@
     (pin "2")
   )
+  (symbol (lib_id "power:GND") (at 307.34 121.92 0) (unit 1)
+    (in_bom yes) (on_board yes)
+    (property "Reference" "#PWR047" (id 0) (at 307.34 128.27 0)
+      (effects (font (size 1.27 1.27)) hide)
+    )
+    (property "Value" "GND" (id 1) (at 307.467 126.3142 0))
+    (property "Footprint" "" (id 2) (at 307.34 121.92 0)
+      (effects (font (size 1.27 1.27)) hide)
+    )
+    (property "Datasheet" "" (id 3) (at 307.34 121.92 0)
+      (effects (font (size 1.27 1.27)) hide)
+    )
+    (pin "1")
+  )
   (symbol (lib_id "Device:R_Small") (at 278.13 120.65 0) (unit 1)
     (in_bom yes) (on_board yes)
@@
     (in_bom yes) (on_board yes)
     (property "Reference" "U7" (id 0) (at 325.12 45.72 0))
-    (property "Value" "TL074" (id 1) (at 326.39 48.26 0))
+    (property "Value" "MCP6004" (id 1) (at 326.39 48.26 0))
     (property "Footprint" "Package_SO:SOIC-14_3.9x8.7mm_P1.27mm" (id 2) (at 320.04 48.26 0)
       (effects (font (size 1.27 1.27)) hide)
@@
     (pin "2")
   )
+  (symbol (lib_id "power:GND") (at 307.34 101.6 0) (unit 1)
+    (in_bom yes) (on_board yes)
+    (property "Reference" "#PWR042" (id 0) (at 307.34 107.95 0)
+      (effects (font (size 1.27 1.27)) hide)
+    )
+    (property "Value" "GND" (id 1) (at 307.467 105.9942 0))
+    (property "Footprint" "" (id 2) (at 307.34 101.6 0)
+      (effects (font (size 1.27 1.27)) hide)
+    )
+    (property "Datasheet" "" (id 3) (at 307.34 101.6 0)
+      (effects (font (size 1.27 1.27)) hide)
+    )
+    (pin "1")
+  )
   (symbol (lib_id "Amplifier_Operational:TL074") (at 321.31 36.83 0) (unit 2)
     (in_bom yes) (on_board yes)
     (property "Reference" "U7" (id 0) (at 325.12 31.75 0))
-    (property "Value" "TL074" (id 1) (at 326.39 34.29 0))
+    (property "Value" "MCP6004" (id 1) (at 326.39 34.29 0))
     (property "Footprint" "Package_SO:SOIC-14_3.9x8.7mm_P1.27mm" (id 2) (at 320.04 34.29 0)
       (effects (font (size 1.27 1.27)) hide)
@@
       (reference "#PWR041") (unit 1) (value "+5V") (footprint "")
     )
+    (path "/e6b53734-fadc-469f-a149-b12c718f7663"
+      (reference "#PWR042") (unit 1) (value "GND") (footprint "")
+    )
     (path "/00000000-0000-0000-0000-00005fe8cc6f"
       (reference "#PWR043") (unit 1) (value "+5VA") (footprint "")
@@
       (reference "#PWR046") (unit 1) (value "GND") (footprint "")
     )
+    (path "/be5be810-6cb5-47d7-80b2-8d32577bb502"
+      (reference "#PWR047") (unit 1) (value "GND") (footprint "")
+    )
     (path "/00000000-0000-0000-0000-00005ff688bd"
       (reference "#PWR049") (unit 1) (value "GND") (footprint "")
@@
       (reference "R31") (unit 1) (value "10K") (footprint "Resistor_SMD:R_0805_2012Metric")
     )
+    (path "/2d99624c-eea0-4021-a743-3979b717b79b"
+      (reference "R32") (unit 1) (value "2M") (footprint "Resistor_SMD:R_0805_2012Metric")
+    )
+    (path "/b3ff9613-e29d-4548-8e02-d4434399cd02"
+      (reference "R33") (unit 1) (value "2M") (footprint "Resistor_SMD:R_0805_2012Metric")
+    )
     (path "/71e207d5-050e-4c05-83e1-34abe240229b"
       (reference "RV1") (unit 1) (value "10K") (footprint "Potentiometer_THT:Potentiometer_Alps_RK097_Dual_Horizontal")
@@
     )
     (path "/0027c752-1087-454b-a5ca-3bd0fd178a9c"
-      (reference "U7") (unit 1) (value "TL074") (footprint "Package_SO:SOIC-14_3.9x8.7mm_P1.27mm")
+      (reference "U7") (unit 1) (value "MCP6004") (footprint "Package_SO:SOIC-14_3.9x8.7mm_P1.27mm")
     )
     (path "/e7ded170-bc98-4835-a4f0-c3931de18f6a"
-      (reference "U7") (unit 2) (value "TL074") (footprint "Package_SO:SOIC-14_3.9x8.7mm_P1.27mm")
+      (reference "U7") (unit 2) (value "MCP6004") (footprint "Package_SO:SOIC-14_3.9x8.7mm_P1.27mm")
     )
     (path "/d5bd7ff8-5fcc-4fa9-9437-42f42f96d761"
-      (reference "U7") (unit 3) (value "TL074") (footprint "Package_SO:SOIC-14_3.9x8.7mm_P1.27mm")
+      (reference "U7") (unit 3) (value "MCP6004") (footprint "Package_SO:SOIC-14_3.9x8.7mm_P1.27mm")
     )
     (path "/a25e5a92-4b29-4a02-8370-0042d42d9b8c"
-      (reference "U7") (unit 4) (value "TL074") (footprint "Package_SO:SOIC-14_3.9x8.7mm_P1.27mm")
+      (reference "U7") (unit 4) (value "MCP6004") (footprint "Package_SO:SOIC-14_3.9x8.7mm_P1.27mm")
     )
     (path "/b1053bb8-795f-46e0-8300-62f7b6a71e98"
-      (reference "U7") (unit 5) (value "TL074") (footprint "Package_SO:SOIC-14_3.9x8.7mm_P1.27mm")
+      (reference "U7") (unit 5) (value "MCP6004") (footprint "Package_SO:SOIC-14_3.9x8.7mm_P1.27mm")
     )
     (path "/8770a895-9aed-427a-86ef-c9fa5bcd4b77"
